Commit message: port to ros2

File: resources/double_integrator/urdf/double_integrator.urdf (robot description, URDF)
Before this commit: robot double_integrator, 3 links, 2 joints
Links:
- link slideBar: mass 0.1 -> None

File: resources/quadrotor/urdf/quadrotor.urdf (robot description, URDF)
Before this commit: robot quadrotor, 1 links, 0 joints
Links:
- link base: geometry collision cylinder length=.1 radius=.3; visual mesh filename=package://ocs2_robotic_assets/resources/quadrotor/meshes/qu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 scale=.4 .4 .4
