Commit message: Update URDF to SVD URDF.

File: resources/mobile_manipulator/kuka/urdf/kuka.urdf (robot description, URDF)
Before this commit: robot med7, 12 links, 11 joints
Links:
- link link_drillbit: geometry collision cylinder length=0.031 radius=0.0032; visual cylinder length=0.031 radius=0.0032
- link link_ee: geometry collision cylinder length=0.22 radius=0.04; visual mesh filename=package://ocs2_robotic_assets/resources/mobile_manipulator/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 scale=0.001 0.001 0.001
Joints:
- joint joint_drillbit: origin xyz=0 0 0.2 rpy=0 0 0 -> xyz=0 0 0.2285 rpy=0 0 0
- joint joint_tool: origin xyz=0 0 0.0326 rpy=0 0 0 -> xyz=0 0 0.031 rpy=0 0 0
